File: Flight_Computer.kicad_sch (KiCad schematic)
At the start: 59 parts, among them J1 PYRO, J2 PYRO, J3 Conn_01x04, J5 Conn_01x02_Pin, J6 Conn_01x09_Socket, J9 Conn_01x02_Pin, Q1 IRLZ44N, Q2 IRLZ44N, SW2 SW_Push, SW3 SW_Push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

Commit message: Upload final pcb and schematic version
Parts:
- removed R10, R16: 1, Resistor_SMD:R_0805_2012Metric, symbol Device:R
- removed TP13, TP14, TP15, TP16: TestPoint, TestPoint:TestPoint_Pad_D2.0mm, symbol Connector:TestPoint
- added R20, R22: 10K, Resistor_SMD:R_0805_2012Metric, symbol Device:R
- C21, C22, C5, C8: footprint Capacitor_SMD:C_0603_1608Metric -> Capacitor_SMD:C_0805_2012Metric
- C4, C6: footprint Capacitor_SMD:C_0201_0603Metric -> Capacitor_SMD:C_0805_2012Metric
- U1: footprint TLV1117-33CDCY:SOT230P700X180-4N -> Package_TO_SOT_SMD:SOT-223-3_TabPin2
Connections:
- net BARO_INT: now also U2.29 (IO36); no longer U2.15 (IO3)
- net BATT_IN: now also R20.1
- net BUTT_0: now also U2.38 (IO2); no longer U2.30 (IO37)
- net BUZZER: now also U2.39 (IO1); no longer U2.9 (IO16)
- net GND: now also R22.2
- net GPS_EXTINT: now also U2.15 (IO3); no longer U2.29 (IO36)
- net IMU_INT: now also U2.30 (IO37); no longer U2.12 (IO8)
- net PYRO_1: now also U2.9 (IO16); no longer U2.39 (IO1)
- net SENSE_1: now also U2.13 (USB_D-); no longer U2.38 (IO2)
- net at J1.1 (Pin_1): now also Q2.2 (D), R18.2
- net at J2.1 (Pin_1): now also Q1.2 (D), R11.2
- new net BATT_SENSE: R20.2, R22.1, U2.12 (IO8)
- no-connect marks 5 -> 4
Other:
- moved on the sheet: TP10
